Commit message: updated urdf file

File: Path_Planning_ws/src/maze_bot/urdf/maze_bot.urdf (robot description, URDF)
Before this commit: robot maze_bot, 5 links, 4 joints
Links:
- added link camera_link
- link base: mass 5 -> 2; geometry collision mesh filename=package://maze_bot/meshes/base_link.stl; visual mesh filename=package://maze_bot/meshes/base_link.stl
- link caster: mass 1 -> 0.75; geometry collision mesh filename=package://maze_bot/meshes/front_caster.stl; visual mesh filename=package://maze_bot/meshes/front_caster.stl
- link wheel_left: mass 1 -> 0.75; geometry collision mesh filename=package://maze_bot/meshes/wheel_l.stl; visual mesh filename=package://maze_bot/meshes/wheel_l.stl
- link wheel_right: mass 1 -> 0.75; geometry collision mesh filename=package://maze_bot/meshes/wheel_r.stl; visual mesh filename=package://maze_bot/meshes/wheel_r.stl
Joints:
- added joint camera_joint: type fixed, parent base, child camera_link, origin xyz=-0.16 0.0 0.08 rpy=0 0.0 3.14, axis 0.0 0.0 1.0
- joint caster_joint: axis 0.0 0.0 1.0 -> 0 0 1
- joint wheel_left_joint: axis 0.0 1.0 0.0 -> 0.0 1 0; origin xyz=0.09 -0.1 0.04 rpy=0.0 0.0 3.14 -> xyz=0.09 -0.1 0.04 rpy=0 0.0 3.14
- joint wheel_right_joint: axis 0.0 1.0 0.0 -> 0.0 -1.0 0; origin xyz=0.09 0.085 0.04 rpy=0.0 0.0 0.0 -> xyz=0.09 0.085 0.04   rpy=0 0.0 0.0

Commit message: Aded Maze solver node
Fixed bugs in world and launch file added localization logic

File: Path_Planning_ws/src/maze_bot/urdf/maze_bot.urdf (robot description, URDF)
Before this commit: robot maze_bot, 6 links, 5 joints
Links:
- link base: geometry collision mesh filename=package://maze_bot/meshes/Base.stl; visual mesh filename=package://maze_bot/meshes/Base.stl
- link caster: geometry collision mesh filename=package://maze_bot/meshes/Wheel_F.stl; visual mesh filename=package://maze_bot/meshes/Wheel_F.stl
- link wheel_left: geometry collision mesh filename=package://maze_bot/meshes/Wheel_L.stl; visual mesh filename=package://maze_bot/meshes/Wheel_L.stl
- link wheel_right: geometry collision mesh filename=package://maze_bot/meshes/Wheel_R.stl; visual mesh filename=package://maze_bot/meshes/Wheel_R.stl
